File: pytheasFC_0.1.0.kicad_sch (KiCad schematic)
At the start: 73 parts, among them IC1 BMP390, IC2 ATSAMD21G18A-MFT, IC3 MIC24054YJL-TR, IC4 TLV1117LV33DCYR, J10 Conn_01x02, J13 Conn_01x02, J14 Conn_01x02, J15 Conn_01x02, J2 USB_C_Receptacle_USB2.0_14P, J3 TagConnect_NL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

Commit message: update VDDANA net and connections
Parts:
- R1, R10, R11, R12, R13, R2, R3, R4, R5, R6, R7, R8, R9: footprint Capacitor_SMD:C_0402_1005Metric -> Resistor_SMD:R_0402_1005Metric
Connections:
- net VDDANA is gone; now on net +3V3: C1.1, C2.1, IC2.6 (VDDANA)
Other:
- moved on the sheet: C2
Changed lines of the file:
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@@
 	)
 	(junction
-		(at 199.39 105.41)
-		(diameter 0)
-		(color 0 0 0 0)
-	)
-	(junction
 		(at 88.9 179.07)
 		(diameter 0)
@@
 	)
 	(junction
-		(at 199.39 96.52)
-		(diameter 0)
-		(color 0 0 0 0)
-	)
-	(junction
 		(at 236.22 67.31)
 		(diameter 0)
@@
 	)
 	(junction
+		(at 203.2 105.41)
+		(diameter 0)
+		(color 0 0 0 0)
+	)
+	(junction
 		(at 67.31 132.08)
 		(diameter 0)
@@
 	)
 	(junction
+		(at 203.2 86.36)
+		(diameter 0)
+		(color 0 0 0 0)
+	)
+	(junction
+		(at 203.2 96.52)
+		(diameter 0)
+		(color 0 0 0 0)
+	)
+	(junction
 		(at 83.82 38.1)
 		(diameter 0)
@@
 	(wire
 		(pts
+			(xy 203.2 85.09) (xy 203.2 86.36)
+		)
+		(stroke
+			(width 0)
+			(type default)
+		)
+	)
+	(wire
+		(pts
 			(xy 219.71 93.98) (xy 227.33 93.98)
 		)
@@
 	(wire
 		(pts
-			(xy 187.96 96.52) (xy 199.39 96.52)
+			(xy 187.96 96.52) (xy 203.2 96.52)
 		)
 		(stroke
@@
 	(wire
 		(pts
-			(xy 167.64 105.41) (xy 199.39 105.41)
+			(xy 167.64 105.41) (xy 203.2 105.41)
 		)
 		(stroke
@@
 	(wire
 		(pts
-			(xy 187.96 86.36) (xy 199.39 86.36)
+			(xy 187.96 86.36) (xy 203.2 86.36)
 		)
 		(stroke
@@
 	(wire
 		(pts
-			(xy 199.39 86.36) (xy 199.39 87.63)
+			(xy 203.2 86.36) (xy 203.2 87.63)
 		)
 		(stroke
@@
 	(wire
 		(pts
-			(xy 199.39 95.25) (xy 199.39 96.52)
+			(xy 203.2 95.25) (xy 203.2 96.52)
 		)
 		(stroke
@@
 	(wire
 		(pts
-			(xy 199.39 105.41) (xy 199.39 96.52)
+			(xy 203.2 105.41) (xy 203.2 96.52)
 		)
 		(stroke
@@
 	(wire
 		(pts
-			(xy 199.39 105.41) (xy 199.39 106.68)
+			(xy 203.2 105.41) (xy 203.2 106.68)
 		)
 		(stroke
@@
 			)
 		)
-		(property "Footprint" "Capacitor_SMD:C_0402_1005Metric"
+		(property "Footprint" "Resistor_SMD:R_0402_1005Metric"
 			(at 212.852 36.83 90)
 			(effects
@@
 			)
 		)
+		(property "Part Number" ""
+			(at 214.63 36.83 0)
+			(effects
+				(font
+					(size 1.27 1.27)
+				)
+				(hide yes)
+			)
+		)
 		(pin "1"
 		)
@@
 			)
 		)
-		(property "Footprint" "Capacitor_SMD:C_0402_1005Metric"
+		(property "Footprint" "Resistor_SMD:R_0402_1005Metric"
 			(at 270.002 138.43 90)
 			(effects
@@
 			)
 		)
-		(property "Footprint" "Capacitor_SMD:C_0402_1005Metric"
+		(property "Footprint" "Resistor_SMD:R_0402_1005Metric"
 			(at 243.332 99.06 90)
 			(effects
@@
 			)
 		)
-		(property "Footprint" "Capacitor_SMD:C_0402_1005Metric"
+		(property "Footprint" "Resistor_SMD:R_0402_1005Metric"
 			(at 193.802 26.67 90)
 			(effects
@@
 			)
 		)
+		(property "Part Number" ""
+			(at 195.58 26.67 0)
+			(effects
+				(font
+					(size 1.27 1.27)
+				)
+				(hide yes)
+			)
+		)
 		(pin "1"
 		)
@@
 			)
 		)
-		(property "Footprint" "Capacitor_SMD:C_0402_1005Metric"
+		(property "Footprint" "Resistor_SMD:R_0402_1005Metric"
 			(at 32.258 161.29 90)
 			(effects
@@
 			)
 		)
-		(property "Footprint" "Capacitor_SMD:C_0402_1005Metric"
+		(property "Footprint" "Resistor_SMD:R_0402_1005Metric"
 			(at 76.962 170.18 90)
 			(effects
@@
 			)
 		)
-		(property "Footprint" "Capacitor_SMD:C_0402_1005Metric"
+		(property "Footprint" "Resistor_SMD:R_0402_1005Metric"
 			(at 103.632 69.85 90)
 			(effects
@@
 	(symbol
 		(lib_id "power:GND")
-		(at 199.39 106.68 0)
+		(at 203.2 106.68 0)
 		(unit 1)
 		(exclude_from_sim no)
@@
 		(dnp no)
 		(property "Reference" "#PWR01"
-			(at 199.39 113.03 0)
+			(at 203.2 113.03 0)
 			(effects
 				(font
@@
 		)
 		(property "Value" "GND"
-			(at 199.39 111.76 0)
+			(at 203.2 111.76 0)
 			(effects
 				(font
@@
 		)
 		(property "Footprint" ""
-			(at 199.39 106.68 0)
+			(at 203.2 106.68 0)
 			(effects
 				(font
@@
 		)
 		(property "Datasheet" ""
-			(at 199.39 106.68 0)
+			(at 203.2 106.68 0)
 			(effects
 				(font
@@
 		)
 		(property "Description" "Power symbol creates a global label with name \"GND\" , ground"
-			(at 199.39 106.68 0)
+			(at 203.2 106.68 0)
 			(effects
 				(font
@@
 		)
 		(property "Price for one" ""
-			(at 199.39 106.68 0)
+			(at 203.2 106.68 0)
 			(effects
 				(font
@@
 			)
 		)
-		(property "Footprint" "Capacitor_SMD:C_0402_1005Metric"
+		(property "Footprint" "Resistor_SMD:R_0402_1005Metric"
 			(at 198.882 54.61 90)
 			(effects
@@
 	)
 	(symbol
+		(lib_id "power:+3V3")
+		(at 203.2 85.09 0)
+		(unit 1)
+		(exclude_from_sim no)
+		(in_bom yes)
+		(on_board yes)
+		(dnp no)
+		(property "Reference" "#PWR034"
+			(at 203.2 88.9 0)
+			(effects
+				(font
+					(size 1.27 1.27)
+				)
+				(hide yes)
+			)
+		)
+		(property "Value" "+3V3"
+			(at 202.946 81.534 0)
+			(effects
+				(font
+					(size 1.27 1.27)
+				)
+			)
+		)
+		(property "Footprint" ""
+			(at 203.2 85.09 0)
+			(effects
+				(font
+					(size 1.27 1.27)
+				)
+				(hide yes)
+			)
+		)
+		(property "Datasheet" ""
+			(at 203.2 85.09 0)
+			(effects
+				(font
+					(size 1.27 1.27)
+				)
+				(hide yes)
+			)
+		)
+		(property "Description" "Power symbol creates a global label with name \"+3V3\""
+			(at 203.2 85.09 0)
+			(effects
+				(font
+					(size 1.27 1.27)
+				)
+				(hide yes)
+			)
+		)
+		(pin "1"
+		)
+		(instances
+			(project "pytheasFC_0.1.0"
+				(path "/a3c366f5-898b-4b05-b602-549e243c6fbe"
+					(reference "#PWR034")
+					(unit 1)
+				)
+			)
+		)
+	)
+	(symbol
 		(lib_id "Device:C")
 		(at 52.07 68.58 0)
@@
 			)
 		)
-		(property "Footprint" "Capacitor_SMD:C_0402_1005Metric"
+		(property "Footprint" "Resistor_SMD:R_0402_1005Metric"
 			(at 244.348 99.06 90)
 			(effects
@@
 			)
 		)
-		(property "Footprint" "Capacitor_SMD:C_0402_1005Metric"
+		(property "Footprint" "Resistor_SMD:R_0402_1005Metric"
 			(at 199.898 54.61 90)
 			(effects
@@
 			)
 		)
-		(property "Footprint" "Capacitor_SMD:C_0402_1005Metric"
+		(property "Footprint" "Resistor_SMD:R_0402_1005Metric"
 			(at 76.962 160.02 90)
 			(effects
@@
 	(symbol
 		(lib_id "Device:C")
-		(at 199.39 91.44 0)
+		(at 203.2 91.44 0)
 		(unit 1)
 		(exclude_from_sim no)
@@
 		(dnp no)
 		(property "Reference" "C2"
-			(at 202.184 90.17 0)
+			(at 205.994 90.17 0)
 			(effects
 				(font
@@
 		)
 		(property "Value" "10uF"
-			(at 202.184 92.71 0)
+			(at 205.994 92.71 0)
 			(effects
 				(font
@@
 		)
 		(property "Footprint" "Capacitor_SMD:C_0805_2012Metric"
-			(at 200.3552 95.25 0)
+			(at 204.1652 95.25 0)
 			(effects
 				(font
@@
 		)
 		(property "Datasheet" "~"
-			(at 199.39 91.44 0)
+			(at 203.2 91.44 0)
 			(effects
 				(font
@@
 		)
 		(property "Description" "Unpolarized capacitor"
-			(at 199.39 91.44 0)
+			(at 203.2 91.44 0)
 			(effects
 				(font
@@
 		)
 		(property "Price for one" ""
-			(at 199.39 91.44 0)
+			(at 203.2 91.44 0)
 			(effects
 				(font
@@
 		)
 		(property "Distributer Link" ""
-			(at 199.39 91.44 0)
+			(at 203.2 91.44 0)
 			(effects
 				(font
@@
 		)
 		(property "Part #" ""
-			(at 199.39 91.44 0)
+			(at 203.2 91.44 0)
 			(effects
 				(font
@@
 			)
 		)
-		(property "Footprint" "Capacitor_SMD:C_0402_1005Metric"
+		(property "Footprint" "Resistor_SMD:R_0402_1005Metric"
 			(at 217.932 101.6 90)
 			(effects
@@
 			)
 		)
-		(property "Footprint" "Capacitor_SMD:C_0402_1005Metric"
+		(property "Footprint" "Resistor_SMD:R_0402_1005Metric"
 			(at 16.002 154.94 90)
 			(effects
